File: redstone_dust/redstone.kicad_sch (KiCad schematic)
At the start: 69 parts, among them J1 1x4_Pogo, J2 1x4_Pogo, J3 1x4_Pogo, J4 1x4_Pogo, J5 1x4_Pogo, J6 1x4_Pogo, J7 1x4_Pogo, J8 1x4_Pogo, J9 2.54mm_ProgrammingPin, Q1 BC108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

Commit message: add more traces, almost done
Parts:
- added C6: 0.1uF, SamacSys_Parts:CAPC2012X140N, symbol SamacSys_Parts:C0805F104K1RACAUTO
- added C7: 1uF, SamacSys_Parts:CAPC0603X33N, symbol SamacSys_Parts:GRM033D70E105ME15D
Connections:
- net E_RX: now also U1.29 (GPIO18); no longer U1.31 (GPIO20)
- net E_TX: now also U1.30 (GPIO19); no longer U1.32 (GPIO21)
- net GND: now also J9.1 (Pin_1), C6.2, C7.2; no longer J9.4 (Pin_4)
- net N_RX: now also U1.37 (GPIO25); no longer U1.36 (GPIO24)
- net N_TX: now also U1.36 (GPIO24); no longer U1.37 (GPIO25)
- net S_RX: now also U1.17 (GPIO14); no longer U1.11 (GPIO8)
- net S_TX: now also U1.16 (GPIO13); no longer U1.12 (GPIO9)
- net at SW1.2 (B), U1.26 (RUN): now also J9.4 (Pin_4), C6.1, C7.1; no longer J9.1 (Pin_1)
- net at J9.2 (Pin_2): now also U1.25 (SWD); no longer U1.24 (SWCLK)
- net at J9.3 (Pin_3): now also U1.24 (SWCLK); no longer U1.25 (SWD)
- net at R20.2: now also U1.15 (GPIO12); no longer U1.27 (GPIO16)
Other:
- moved on the sheet: J9
