File: redstone_block/redstone_block.kicad_pcb (KiCad board)
At the start: 2 copper layers, 40 x 40 mm, 44 parts, among them J1 1x4_Pogo, J2 1x4_Pogo, J3 1x4_Pogo, J4 1x4_Pogo, J5 1x4_Pogo, J6 1x4_Pogo, J7 1x4_Pogo, J8 1x4_Pogo, J9 2.54mm_ProgrammingPin, SW1 SW_Push_Open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

Commit message: remove unecessary silkscreen markings on redstone block
Parts:
- renumbered R17 to 100k
Other:
- board text removed: "+"
Changed lines of the file:
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@@
 		(descr "1210 (3225 Metric)")
 		(tags "Resistor")
-		(property "Reference" "R17"
+		(property "Reference" "100k"
 			(at 2 3.5 180)
 			(layer "F.SilkS")
@@
 		(layer "Edge.Cuts")
 	)
-	(gr_text "+"
-		(at 133.5 61 0)
-		(layer "F.SilkS")
-		(effects
-			(font
-				(size 1 1)
-				(thickness 0.15)
-				(bold yes)
-			)
-		)
-	)
 	(gr_text "PGM"
